File: PB SAO.kicad_pcb (KiCad board)
At the start: 2 copper layers, 52 x 150.4 mm, 15 parts, among them P1 SAO_1

Commit message: Add files via upload
V2 including Mag0r's edits.
Parts:
- removed >NAME (x4): >VALUE, adafruit:sidebendLED3MM
- removed P1: SAO_1, adafruit:SAO_Header_6-Pin_Oval_AltPins
- removed REF** (x4): 1206, digikey-footprints:1206
- removed REF**: Switch_Tactile_THT_6x6mm_MJTP1230, digikey-footprints:Switch_Tactile_THT_6x6mm_MJTP1230
- removed Ref**: Battery Holder, adafruit:CoinCellBatt2032
- removed S1: SMDButton4x4x1.5elkei, adafruit:SMDButton4x4x1.5elkei
- removed Slide Switch: SK12D07 Slide Switch Through Hole ELKEI, adafruit:SK12D07 Slide Switch Through Hole ELKEI
- added D1: LED, LED_SMD:LED_0805_2012Metric_Pad1.15x1.40mm_HandSolder, B.Cu at (89.2, 36.3)
- added D2: LED, LED_SMD:LED_0805_2012Metric_Pad1.15x1.40mm_HandSolder, B.Cu at (89.1, 53.1)
- added D3: LED, LED_SMD:LED_0805_2012Metric_Pad1.15x1.40mm_HandSolder, B.Cu at (89.2, 95.2)
- added D4: LED, LED_SMD:LED_0805_2012Metric_Pad1.15x1.40mm_HandSolder, B.Cu at (89.8, 137.0)
- added D5: LED, LED_THT:LED_D3.0mm, B.Cu at (87.9, 39.6)
- added D6: LED, LED_THT:LED_D3.0mm, B.Cu at (87.9, 55.4)
- added D7: LED, LED_THT:LED_D3.0mm, B.Cu at (87.9, 98.8)
- added D8: LED, LED_THT:LED_D3.0mm, B.Cu at (88.5, 140.3)
- added G***: LOGO, F.Mask_g842, F.Cu at (108.0, 155.0)
- added G***: LOGO, F.Cu_g824, F.Cu at (111.8, 98.5)
- added G***: LOGO, F.SilkS_g838, F.Cu at (116.1, 98.9)
- added G***: LOGO, F.Mask_g842, F.Cu at (115.7, 99.1)
- added G***: LOGO, F.Mask_g842, F.Cu at (111.8, 98.6)
- added H1: MountingHole, MountingHole:MountingHole_3mm, F.Cu at (141.3, 145.8)
- added J1: SAO_F, Connector_PinHeader_2.54mm:PinHeader_2x03_P2.54mm_Vertical, F.Cu at (153.3, 171.1)
- added J2: SAO_F, Connector_PinHeader_2.54mm:PinHeader_2x03_P2.54mm_Vertical, B.Cu at (99.4, 168.7)
- added Q1: 2N7002, Package_TO_SOT_SMD:SOT-23_Handsoldering, B.Cu at (85.5, 147.2)
- added Q2: 2N7002, Package_TO_SOT_THT:TO-92, B.Cu at (92.7, 147.0)
- added SW1: SW_Push, Button_Switch_THT:SW_PUSH_6mm, F.Cu at (86.0, 103.3)
- added SW2: SW_Push, Button_Switch_SMD:SW_Push_1P1T_NO_6x6mm_H9.5mm, F.Cu at (89.3, 105.6)
- BT1: value BATTERY-20MM_SMD_4LEGS -> CR2032; footprint BatteryHolder_Keystone_3034_1x20mm -> Battery:BatteryHolder_Keystone_3034_1x20mm
- moved G*** 26.5 mm to (119.9, 151.8)
- moved BT1 18.6 mm to (141.3, 159.3), turned to 180 degrees
Connections:
- BT1 pad 1: (no net) -> +3V3
- BT1 pad 2: (no net) -> GND
Routing:
- net (no net): track 355.8 -> 2.03 mm, vias 1 -> 0
- net /VCC: track 0.00 -> 181.1 mm
- net Net-(D1-Pad1): track 0.00 -> 139.6 mm
- net GND: track 0.00 -> 70.3 mm
- net /IO_high: track 0.00 -> 58.4 mm, vias 0 -> 1
- net +3V3: track 0.00 -> 48.9 mm
- net Net-(J2-Pad5): track 0.00 -> 9.12 mm
- net Net-(J1-Pad5): track 0.00 -> 2.54 mm
Other:
- board size 52 x 150.4 mm -> 97.9 x 150.9 mm
- board text added: "+"
- board text added: "-"
- board text added: "LinuxConf 2022"
- board text added: "THE PARTY BUTTON"
